Commit message: svan m1 training done

File: resources/robots/svan_m2/urdf/svan_urdf_package_inertia.urdf (robot description, URDF)
Before this commit: robot svan_urdf_package, 17 links, 16 joints
Links:
- added link base; visual box size=0.001 0.001 0.001
- link base_link: mass 2.99710872609609 -> 4.713
- link fl_abd_l: mass 0.547089526327068 -> 0.696
- link fl_hip_l: mass 0.147108571121327 -> 1.013
- link fl_knee_a: mass 0.122422228142348 -> 0.166
- link fr_abd_l: mass 0.547089526327116 -> 0.696
- link fr_hip_l: mass 0.147108571121328 -> 1.013
- link fr_knee_l: mass 0.122422228142348 -> 0.166
- link rl_abd_l: mass 0.547089526327067 -> 0.696
- link rl_hip_l: mass 0.147108560926126 -> 1.013
- link rl_knee_l: mass 0.122422317176859 -> 0.166
- link rr_abd_l: mass 0.547089526327114 -> 0.696
- link rr_hip_l: mass 0.147108571121328 -> 1.013
- link rr_knee_l: mass 0.122422246876929 -> 0.166
Joints:
- added joint floating_base: type fixed, parent base, child base_link, origin xyz=0 0 0 rpy=0 0 0
