Commit message: urdf updated

File: resources/robots/svan_m2/urdf/svan_urdf_package.urdf (robot description, URDF)
Before this commit: robot svan_urdf_package, 17 links, 16 joints
Links:
- removed link base_link
- removed link fl_abd_l
- removed link fl_hip_l
- removed link foot_FL
- removed link foot_FR
- removed link foot_RL
- removed link foot_RR
- removed link fr_abd_l
- removed link fr_hip_l
- removed link fr_knee_l
- removed link rl_abd_l
- removed link rl_hip_l
- removed link rl_knee_l
- removed link rr_abd_l
- removed link rr_hip_l
- removed link rr_knee_l
- added link FL_foot, mass 0.025; collision sphere radius=0.01; visual sphere radius=0.01
- added link FL_hip, mass 0.547089526327068; collision mesh filename=../meshes/fl_abd_l.STL; visual mesh filename=../meshes/fl_abd_l.STL
- added link FL_thigh, mass 0.147108571121327; collision mesh filename=../meshes/fl_hip_l.STL; visual mesh filename=../meshes/fl_hip_l.STL
- added link FR_calf, mass 0.122422228142348; collision mesh filename=../meshes/fr_knee_l.STL; visual mesh filename=../meshes/fr_knee_l.STL
- added link FR_foot, mass 0.025; collision sphere radius=0.01; visual sphere radius=0.01
- added link FR_hip, mass 0.547089526327116; collision mesh filename=../meshes/fr_abd_l.STL; visual mesh filename=../meshes/fr_abd_l.STL
- added link FR_thigh, mass 0.147108571121328; collision mesh filename=../meshes/fr_hip_l.STL; visual mesh filename=../meshes/fr_hip_l.STL
- added link RL_calf, mass 0.122422317176859; collision mesh filename=../meshes/rl_knee_l.STL; visual mesh filename=../meshes/rl_knee_l.STL
- added link RL_foot, mass 0.025; collision sphere radius=0.01; visual sphere radius=0.01
- added link RL_hip, mass 0.547089526327067; collision mesh filename=../meshes/rl_abd_l.STL; visual mesh filename=../meshes/rl_abd_l.STL
- added link RL_thigh, mass 0.147108560926126; collision mesh filename=../meshes/rl_hip_l.STL; visual mesh filename=../meshes/rl_hip_l.STL
- added link RR_calf, mass 0.122422246876929; collision mesh filename=../meshes/rr_knee_l.STL; visual mesh filename=../meshes/rr_knee_l.STL
- added link RR_foot, mass 0.025; collision sphere radius=0.01; visual sphere radius=0.01
- added link RR_hip, mass 0.547089526327114; collision mesh filename=../meshes/rr_abd_l.STL; visual mesh filename=../meshes/rr_abd_l.STL
- added link RR_thigh, mass 0.147108571121328; collision mesh filename=../meshes/rr_hip_l.STL; visual mesh filename=../meshes/rr_hip_l.STL
- added link base; visual box size=0.001 0.001 0.001
- added link trunk, mass 2.99710872609609; collision mesh filename=../meshes/torso_link.STL; visual mesh filename=../meshes/torso_link.STL
Joints:
- removed joint fl_abd_j
- removed joint fl_dummy_j
- removed joint fl_hip_j
- removed joint fl_knee_j
- removed joint fr_abd_j
- removed joint fr_dummy_j
- removed joint fr_hip_j
- removed joint fr_knee_j
- removed joint rl_abd_j
- removed joint rl_dummy_j
- removed joint rl_hip_j
- removed joint rl_knee_j
- removed joint rr_abd_j
- removed joint rr_dummy_j
- removed joint rr_hip_j
- removed joint rr_knee_j
- added joint FL_calf_joint: type revolute, parent FL_thigh, child fl_knee_a, origin xyz=0.0041389 -0.01 -0.16494 rpy=0 0 0, axis 0 1 0, limit lower=-3 upper=3 effort=100 velocity=100
- added joint FL_foot_fixed: type fixed, parent fl_knee_a, child FL_foot, origin xyz=-0.026618 0 -0.16693 rpy=0 0 0
- added joint FL_hip_joint: type revolute, parent trunk, child FL_hip, origin xyz=0.20368 0.06 0 rpy=0 0 0, axis 1 0 0, limit lower=-3 upper=3 effort=100 velocity=100
- added joint FL_thigh_joint: type revolute, parent FL_hip, child FL_thigh, origin xyz=0.043 0.07525 0 rpy=0 0 0, axis 0 1 0, limit lower=-3 upper=3 effort=100 velocity=100
- added joint FR_calf_joint: type revolute, parent FR_thigh, child FR_calf, origin xyz=0.0041389 0.01 -0.16494 rpy=0 0 0, axis 0 1 0, limit lower=-3 upper=3 effort=100 velocity=100
- added joint FR_foot_fixed: type fixed, parent FR_calf, child FR_foot, origin xyz=-0.026457 0 -0.16693 rpy=0 0 0
- added joint FR_hip_joint: type revolute, parent trunk, child FR_hip, origin xyz=0.20368 -0.06 0 rpy=0 0 0, axis 1 0 0, limit lower=-3 upper=3 effort=100 velocity=100
- added joint FR_thigh_joint: type revolute, parent FR_hip, child FR_thigh, origin xyz=0.043 -0.07525 0 rpy=0 0 0, axis 0 1 0, limit lower=-3 upper=3 effort=100 velocity=100
- added joint RL_calf_joint: type revolute, parent RL_thigh, child RL_calf, origin xyz=-0.0038618 -0.01 -0.16493 rpy=0 0 0, axis 0 1 0, limit lower=-3 upper=3 effort=100 velocity=100
- added joint RL_foot_fixed: type fixed, parent RL_calf, child RL_foot, origin xyz=-0.0185 0 -0.16802 rpy=0 0 0
- added joint RL_hip_joint: type revolute, parent trunk, child RL_hip, origin xyz=-0.20482 0.06 0 rpy=0 0 0, axis 1 0 0, limit lower=-3 upper=3 effort=100 velocity=100
- added joint RL_thigh_joint: type revolute, parent RL_hip, child RL_thigh, origin xyz=-0.043 0.07525 0 rpy=0 0 0, axis 0 1 0, limit lower=-3 upper=3 effort=100 velocity=100
- added joint RR_calf_joint: type revolute, parent RR_thigh, child RR_calf, origin xyz=-0.0038618 0.01 -0.16493 rpy=0 0 0, axis 0 1 0, limit lower=-3 upper=3 effort=100 velocity=100
- added joint RR_foot_fixed: type fixed, parent RR_calf, child RR_foot, origin xyz=-0.018339 0 -0.16802 rpy=0 0 0
- added joint RR_hip_joint: type revolute, parent trunk, child RR_hip, origin xyz=-0.20482 -0.06 0 rpy=0 0 0, axis 1 0 0, limit lower=-3 upper=3 effort=100 velocity=100
- added joint RR_thigh_joint: type revolute, parent RR_hip, child RR_thigh, origin xyz=-0.043 -0.07525 0 rpy=0 0 0, axis 0 1 0, limit lower=-3 upper=3 effort=100 velocity=100
- added joint floating_base: type fixed, parent base, child trunk, origin xyz=0 0 0 rpy=0 0 0

Commit message: urdf updated

File: resources/robots/svan_m2/urdf/svan_urdf_package.urdf (robot description, URDF)
Before this commit: robot svan_urdf_package, 18 links, 17 joints
Links:
- removed link fl_knee_a
- added link FL_calf, mass 0.122422228142348; collision mesh filename=../meshes/fl_knee_a.STL; visual mesh filename=../meshes/fl_knee_a.STL
Joints:
- joint FL_calf_joint: child fl_knee_a -> FL_calf; limit lower=-3 upper=3 effort=100 velocity=100 -> lower=-2.69653369433 upper=-0.916297857297 effort=55 velocity=28.6
- joint FL_foot_fixed: parent fl_knee_a -> FL_calf
- joint FL_hip_joint: limit lower=-3 upper=3 effort=100 velocity=100 -> lower=-0.802851455917 upper=0.802851455917 effort=20 velocity=52.4
- joint FL_thigh_joint: limit lower=-3 upper=3 effort=100 velocity=100 -> lower=-1.0471975512 upper=4.18879020479 effort=55 velocity=28.6
- joint FR_calf_joint: limit lower=-3 upper=3 effort=100 velocity=100 -> lower=-2.69653369433 upper=-0.916297857297 effort=55 velocity=28.6
- joint FR_hip_joint: limit lower=-3 upper=3 effort=100 velocity=100 -> lower=-0.8 upper=0.8 effort=20 velocity=52.4
- joint FR_thigh_joint: limit lower=-3 upper=3 effort=100 velocity=100 -> lower=-1.0471975512 upper=4.18879020479 effort=55 velocity=28.6
- joint RL_calf_joint: limit lower=-3 upper=3 effort=100 velocity=100 -> lower=-2.69653369433 upper=-0.916297857297 effort=55 velocity=28.6
- joint RL_hip_joint: limit lower=-3 upper=3 effort=100 velocity=100 -> lower=-0.802851455917 upper=0.802851455917 effort=20 velocity=52.4
- joint RL_thigh_joint: limit lower=-3 upper=3 effort=100 velocity=100 -> lower=-1.0471975512 upper=4.18879020479 effort=55 velocity=28.6
- joint RR_calf_joint: limit lower=-3 upper=3 effort=100 velocity=100 -> lower=-2.69653369433 upper=-0.916297857297 effort=55 velocity=28.6
- joint RR_hip_joint: limit lower=-3 upper=3 effort=100 velocity=100 -> lower=-0.802851455917 upper=0.802851455917 effort=20 velocity=52.4
- joint RR_thigh_joint: limit lower=-3 upper=3 effort=100 velocity=100 -> lower=-1.0471975512 upper=4.18879020479 effort=55 velocity=28.6
